File: PCB/Hackpad.kicad_pcb (KiCad board)
At the start: 2 copper layers, 67.2 x 84.7 mm, 36 parts, among them SW1 SW_Push, SW10 RotaryEncoder_Switch, SW2 SW_Push, SW3 SW_Push, SW4 SW_Push, SW5 SW_Push, SW6 SW_Push, SW7 SW_Push, SW8 SW_Push, SW9 SW_Push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

Commit message: Add files via upload
Parts:
- removed R1: 47k, Resistor_THT:R_Axial_DIN0207_L6.3mm_D2.5mm_P10.16mm_Horizontal
- removed R2: 100k, Resistor_THT:R_Axial_DIN0207_L6.3mm_D2.5mm_P10.16mm_Horizontal
Connections:
- SW10 pad S1: Net-(U1-GPIO3/MOSI) -> unconnected-(SW10-PadS1)
- SW10 pad S2: GND -> unconnected-(SW10-PadS2)
- U1 pad 1: Net-(U1-GPIO26/ADC0/A0) -> A
- U1 pad 11: Net-(U1-GPIO3/MOSI) -> B
Routing:
- net Net-(U1-GPIO3/MOSI): track 37.5 -> 0.00 mm
- net Net-(U1-GPIO26/ADC0/A0): track 33.1 -> 0.00 mm, vias 1 -> 0
- net B: track 33.9 -> 22.1 mm
- net A: track 26.7 -> 25.9 mm, vias 0 -> 1
