File: PCB/Hackpad.kicad_sch (KiCad schematic)
At the start: 32 parts, among them SW1 SW_Push, SW10 RotaryEncoder_Switch, SW2 SW_Push, SW3 SW_Push, SW4 SW_Push, SW5 SW_Push, SW6 SW_Push, SW7 SW_Push, SW8 SW_Push, SW9 SW_Push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

Commit message: Add files via upload
Parts:
- removed R1: 47k, Resistor_THT:R_Axial_DIN0207_L6.3mm_D2.5mm_P10.16mm_Horizontal, symbol Device:R
- removed R2: 100k, Resistor_THT:R_Axial_DIN0207_L6.3mm_D2.5mm_P10.16mm_Horizontal, symbol Device:R
- OLED1: value ~ -> (none)
Connections:
- net A: now also U1.1 (GPIO26/ADC0/A0)
- net B: now also U1.11 (GPIO3/MOSI)
- net GND: no longer SW10.S2
- net at SW10.S1: no longer U1.11 (GPIO3/MOSI)
- no-connect marks 1 -> 3
